File: Motor_Control_Board/Motor_control_Board.kicad_sch (KiCad schematic)
At the start: 0 parts

Commit message: Minor updates: V0.9
Other:
- sheet Motors renamed Motor Driver
Changed lines of the file:
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@@
 			(color 0 0 0 0.0000)
 		)
-		(property "Sheetname" "Motors"
+		(property "Sheetname" "Motor Driver"
 			(at 24.384 63.246 0)
 			(effects
