File: Motor_Control_Board/Power.kicad_sch (KiCad schematic)
At the start: 33 parts, among them J3 Conn_01x02, Q8 PXN012-60QLJ, U3 MAX17643ATC+, U4 LM74610QDGKRQ1, U5 ADP3338AKCZ-3.3-RL

Commit message: Minor updates: V0.9
Parts:
- removed TP1: 5V, TestPoint:TestPoint_Pad_1.5x1.5mm, symbol Connector:TestPoint
- removed TP2: 3.3v, TestPoint:TestPoint_Pad_1.5x1.5mm, symbol Connector:TestPoint
- FB1: PartNum (none) -> ACML-0402-050-T
- L1: PartNum (none) -> XAL5050-103MEC
- Q8: PartNum (none) -> PXN012-60QLJ
- U3: PartNum (none) -> MAX17643ATC+
- U4: PartNum (none) -> LM74610QDGKRQ1
- U5: PartNum (none) -> ADP3338AKCZ-3.3-RL
Other:
- moved on the sheet: H1, H2, H3
