File: Motor_Control_Board/MCU.kicad_sch (KiCad schematic)
At the start: 22 parts, among them J1 TagConnect_TC2030, J4 Encoder, J5 Encoder, SW1 NRST, U1 STM32F103C8Tx, U9 MCP2562FD-E/SN, Y1 ECS-1612MV-080-CN-TR

Commit message: Minor updates: V0.9
Parts:
- added JP1: Jumper_2_Open, Jumper:SolderJumper-2_P1.3mm_Open_TrianglePad1.0x1.5mm, symbol Jumper:Jumper_2_Open
- C30: now not fitted
- J5: value Encoder -> CAN
- R2: footprint (none) -> Resistor_SMD:R_0402_1005Metric; PartNum (none) -> 0402WGF1002TCE
- SW1: PartNum (none) -> NANOT100AS
- U1: PartNum (none) -> STM32F103C8T6
- U9: PartNum (none) -> MCP2562FD-E/SN
- Y1: PartNum (none) -> ECS-1612MV-080-CN-TR
Connections:
- net +5V: now also JP1.1 (A); no longer J5.1 (Pin_1)
- net DRV_FAULT: now reaches U1.40 (PB4)
- new net: J5.1 (Pin_1), JP1.2 (B)
- no-connect marks 19 -> 18
Changed lines of the file:
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@@
 		(at 127 64.77)
 	)
-	(no_connect
-		(at 127 85.09)
-	)
 	(wire
 		(pts
-			(xy 147.32 123.19) (xy 144.78 123.19)
+			(xy 87.63 175.26) (xy 97.79 175.26)
 		)
 		(stroke
@@
 	(wire
 		(pts
-			(xy 31.75 148.59) (xy 44.45 148.59)
+			(xy 147.32 123.19) (xy 144.78 123.19)
 		)
 		(stroke
@@
 	(wire
 		(pts
-			(xy 144.78 120.65) (xy 144.78 123.19)
+			(xy 31.75 148.59) (xy 44.45 148.59)
 		)
 		(stroke
@@
 	(wire
 		(pts
-			(xy 20.32 21.59) (xy 20.32 22.86)
+			(xy 144.78 120.65) (xy 144.78 123.19)
 		)
 		(stroke
@@
 	(wire
 		(pts
-			(xy 96.52 175.26) (xy 97.79 175.26)
+			(xy 20.32 21.59) (xy 20.32 22.86)
 		)
 		(stroke
@@
 	(wire
 		(pts
-			(xy 96.52 173.99) (xy 96.52 175.26)
-		)
-		(stroke
-			(width 0)
-			(type default)
-		)
-	)
-	(wire
-		(pts
 			(xy 142.24 36.83) (xy 142.24 38.1)
 		)
@@
 	(wire
 		(pts
+			(xy 71.12 175.26) (xy 77.47 175.26)
+		)
+		(stroke
+			(width 0)
+			(type default)
+		)
+	)
+	(wire
+		(pts
 			(xy 85.09 153.67) (xy 88.9 153.67)
 		)
@@
 	(wire
 		(pts
+			(xy 125.73 85.09) (xy 127 85.09)
+		)
+		(stroke
+			(width 0)
+			(type default)
+		)
+	)
+	(wire
+		(pts
 			(xy 43.18 146.05) (xy 44.45 146.05)
 		)
@@
 	(wire
 		(pts
+			(xy 71.12 173.99) (xy 71.12 175.26)
+		)
+		(stroke
+			(width 0)
+			(type default)
+		)
+	)
+	(wire
+		(pts
 			(xy 142.24 168.91) (xy 143.51 168.91)
 		)
@@
 		)
 	)
+	(global_label "DRV_FAULT"
+		(shape input)
+		(at 125.73 85.09 180)
+		(fields_autoplaced yes)
+		(effects
+			(font
+				(size 1.27 1.27)
+			)
+			(justify right)
+		)
+		(property "Intersheetrefs" "${INTERSHEET_REFS}"
+			(at 112.6452 85.09 0)
+			(effects
+				(font
+					(size 1.27 1.27)
+				)
+				(justify right)
+				(hide yes)
+			)
+		)
+	)
 	(global_label "ENC_B"
 		(shape input)
@@
 			)
 		)
+		(property "PartNum" "STM32F103C8T6"
+			(at 144.78 80.01 0)
+			(effects
+				(font
+					(size 1.27 1.27)
+				)
+				(hide yes)
+			)
+		)
 		(pin "33"
 		)
@@
 			)
 		)
-		(property "Value" "Encoder"
+		(property "Value" "CAN"
 			(at 105.41 180.3399 0)
 			(effects
@@
 			)
 		)
+		(property "PartNum" "NANOT100AS"
+			(at 41.91 91.44 0)
+			(effects
+				(font
+					(size 1.27 1.27)
+				)
+				(hide yes)
+			)
+		)
 		(pin "2"
 		)
@@
 			)
 		)
+		(property "PartNum" "MCP2562FD-E/SN"
+			(at 44.45 146.05 0)
+			(effects
+				(font
+					(size 1.27 1.27)
+				)
+				(hide yes)
+			)
+		)
 		(pin "8"
 		)
@@
 		(in_bom yes)
 		(on_board yes)
-		(dnp no)
+		(dnp yes)
 		(property "Reference" "C30"
 			(at 126.238 145.542 90)
@@
 	)
 	(symbol
-		(lib_id "power:+24V")
-		(at 96.52 173.99 0)
-		(unit 1)
-		(exclude_from_sim no)
-		(in_bom yes)
-		(on_board yes)
-		(dnp no)
-		(fields_autoplaced yes)
-		(property "Reference" "#PWR083"
-			(at 96.52 177.8 0)
-			(effects
-				(font
-					(size 1.27 1.27)
-				)
-				(hide yes)
-			)
-		)
-		(property "Value" "+5V"
-			(at 96.52 168.91 0)
-			(effects
-				(font
-					(size 1.27 1.27)
-				)
-			)
-		)
-		(property "Footprint" ""
-			(at 96.52 173.99 0)
-			(effects
-				(font
-					(size 1.27 1.27)
-				)
-				(hide yes)
-			)
-		)
-		(property "Datasheet" ""
-			(at 96.52 173.99 0)
-			(effects
-				(font
-					(size 1.27 1.27)
-				)
-				(hide yes)
-			)
-		)
-		(property "Description" "Power symbol creates a global label with name \"+24V\""
-			(at 96.52 173.99 0)
-			(effects
-				(font
-					(size 1.27 1.27)
-				)
-				(hide yes)
-			)
-		)
-		(pin "1"
-		)
-		(instances
-			(project "Motor_control_Board"
-				(path "/8f7cca2f-0bd1-45cd-9991-4ff133d0b08c/a9265767-04bc-48ff-b1a2-646c04a95e03"
-					(reference "#PWR083")
-					(unit 1)
-				)
-			)
-		)
-	)
-	(symbol
 		(lib_id "power:+3.3V")
 		(at 20.32 21.59 0)
@@
 			)
 		)
+		(property "PartNum" "ECS-1612MV-080-CN-TR"
+			(at 83.82 57.15 0)
+			(effects
+				(font
+					(size 1.27 1.27)
+				)
+				(hide yes)
+			)
+		)
 		(pin "4"
 		)
@@
 	)
 	(symbol
+		(lib_id "power:+24V")
+		(at 71.12 173.99 0)
+		(unit 1)
+		(exclude_from_sim no)
+		(in_bom yes)
+		(on_board yes)
+		(dnp no)
+		(fields_autoplaced yes)
+		(property "Reference" "#PWR047"
+			(at 71.12 177.8 0)
+			(effects
+				(font
+					(size 1.27 1.27)
+				)
+				(hide yes)
+			)
+		)
+		(property "Value" "+5V"
+			(at 71.12 168.91 0)
+			(effects
+				(font
+					(size 1.27 1.27)
+				)
+			)
+		)
+		(property "Footprint" ""
+			(at 71.12 173.99 0)
+			(effects
+				(font
+					(size 1.27 1.27)
+				)
+				(hide yes)
+			)
+		)
+		(property "Datasheet" ""
+			(at 71.12 173.99 0)
+			(effects
+				(font
+					(size 1.27 1.27)
+				)
+				(hide yes)
+			)
+		)
+		(property "Description" "Power symbol creates a global label with name \"+24V\""
+			(at 71.12 173.99 0)
+			(effects
+				(font
+					(size 1.27 1.27)
+				)
+				(hide yes)
+			)
+		)
+		(pin "1"
+		)
+		(instances
+			(project "Motor_control_Board"
+				(path "/8f7cca2f-0bd1-45cd-9991-4ff133d0b08c/a9265767-04bc-48ff-b1a2-646c04a95e03"
+					(reference "#PWR047")
+					(unit 1)
+				)
+			)
+		)
+	)
+	(symbol
 		(lib_id "power:+3.3V")
 		(at 101.6 153.67 270)
@@
 			)
 		)
-		(property "Footprint" ""
+		(property "Footprint" "Resistor_SMD:R_0402_1005Metric"
 			(at 40.132 81.28 90)
 			(effects
@@
 			)
 		)
+		(property "PartNum" "0402WGF1002TCE"
+			(at 41.91 81.28 0)
+			(effects
+				(font
+					(size 1.27 1.27)
+				)
+				(hide yes)
+			)
+		)
 		(pin "1"
 		)
@@
 					(unit 1)
 				)
+			)
+		)
+	)
+	(symbol
+		(lib_id "Jumper:Jumper_2_Open")
+		(at 82.55 175.26 0)
+		(unit 1)
+		(exclude_from_sim yes)
+		(in_bom yes)
+		(on_board yes)
+		(dnp no)
+		(fields_autoplaced yes)
+		(property "Reference" "JP1"
+			(at 82.55 168.91 0)
+			(effects
+				(font
+					(size 1.27 1.27)
+				)
+			)
+		)
+		(property "Value" "Jumper_2_Open"
+			(at 82.55 171.45 0)
+			(effects
+				(font
+					(size 1.27 1.27)
+				)
+			)
+		)
+		(property "Footprint" "Jumper:SolderJumper-2_P1.3mm_Open_TrianglePad1.0x1.5mm"
+			(at 82.55 175.26 0)
+			(effects
+				(font
+					(size 1.27 1.27)
+				)
+				(hide yes)
+			)
+		)
+		(property "Datasheet" "~"
+			(at 82.55 175.26 0)
+			(effects
+				(font
+					(size 1.27 1.27)
+				)
+				(hide yes)
+			)
+		)
+		(property "Description" "Jumper, 2-pole, open"
+			(at 82.55 175.26 0)
+			(effects
+				(font
+					(size 1.27 1.27)
+				)
+				(hide yes)
+			)
+		)
+		(pin "1"
+		)
+		(pin "2"
+		)
+		(instances
+			(project ""
+				(path "/8f7cca2f-0bd1-45cd-9991-4ff133d0b08c/a9265767-04bc-48ff-b1a2-646c04a95e03"
+					(reference "JP1")
+					(unit 1)
+				)

Commit message: V0.10 - chnaged Volatge Sensing resistors to enable 48V sensing
Parts:
- C10, C11, C3, C31, C32, C8, R1, R14, R2, R9, SW1, U9, Y1: Supplier (none) -> Mouser
- C30: now fitted
- C5, C6, C7, C9: PartNum GCM1555C1H240FA16J -> C0402C104K4PAC; Supplier (none) -> Mouser
- U1: PartNum STM32F103C8T6 -> STM32F103C8T7; Supplier (none) -> Mouser
Other:
- moved on the sheet: C11, U1, Y1
