File: Motor_Control_Board/Motors.kicad_sch (KiCad schematic)
At the start: 9 parts, among them U2 A4919GLPTR-T

Commit message: Minor updates: V0.9
Parts:
- C24: footprint (none) -> Capacitor_SMD:C_0603_1608Metric; PartNum (none) -> CL10B474KO8NNWC
- D3: value D -> SS12FP; footprint (none) -> Other:DIO_SS12LS_RVG; PartNum (none) -> SS12FP
- U2: PartNum (none) -> A4919GLPTR-T
Changed lines of the file:
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@@
 	(generator "eeschema")
 	(generator_version "8.0")
-	(paper "A4")
+	(paper "A5")
 	(junction
 		(at 115.57 81.28)
@@
 			)
 		)
-		(property "Value" "D"
+		(property "Value" "SS12FP"
 			(at 100.33 22.86 0)
 			(effects
@@
 			)
 		)
-		(property "Footprint" ""
+		(property "Footprint" "Other:DIO_SS12LS_RVG"
 			(at 100.33 26.67 0)
 			(effects
@@
 		)
 		(property "Purchase-URL" ""
+			(at 100.33 26.67 0)
+			(effects
+				(font
+					(size 1.27 1.27)
+				)
+				(hide yes)
+			)
+		)
+		(property "PartNum" "SS12FP "
 			(at 100.33 26.67 0)
 			(effects
@@
 			)
 		)
-		(property "Footprint" ""
+		(property "Footprint" "Capacitor_SMD:C_0603_1608Metric"
 			(at 60.96 53.34 0)
 			(effects
@@
 		)
 		(property "Purchase-URL" ""
+			(at 60.96 53.34 0)
+			(effects
+				(font
+					(size 1.27 1.27)
+				)
+				(hide yes)
+			)
+		)
+		(property "PartNum" "CL10B474KO8NNWC"
 			(at 60.96 53.34 0)
 			(effects
@@
 			(at 105.41 88.9 0)
 			(effects
+				(font
+					(size 1.27 1.27)
+				)
+				(hide yes)
+			)
+		)
+		(property "PartNum" "A4919GLPTR-T"
+			(at 105.41 88.9 0)
+			(effects

Commit message: V0.10 - chnaged Volatge Sensing resistors to enable 48V sensing
Parts:
- C16, C18, C19, C20, C21, C24, D3, U2: Supplier (none) -> Mouser
- C25: PartNum GCM1555C1H240FA16J -> C0402C104K4PAC; Supplier (none) -> Mouser
Changed lines of the file:
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@@
+			)
+		)
+		(property "Supplier" "Mouser"
+			(at 100.33 26.67 0)
+			(effects
+				(font
+					(size 1.27 1.27)
+				)
+				(hide yes)
 			)
 		)
@@
 			)
 		)
+		(property "Supplier" "Mouser"
+			(at 110.49 58.42 0)
+			(effects
+				(font
+					(size 1.27 1.27)
+				)
+				(hide yes)
+			)
+		)
 		(pin "2"
 		)
@@
 			)
 		)
-		(property "PartNum" "GCM1555C1H240FA16J"
+		(property "PartNum" "C0402C104K4PAC"
+			(at 33.02 57.15 0)
+			(effects
+				(font
+					(size 1.27 1.27)
+				)
+				(hide yes)
+			)
+		)
+		(property "Supplier" "Mouser"
 			(at 33.02 57.15 0)
 			(effects
@@
 			)
 		)
+		(property "Supplier" "Mouser"
+			(at 60.96 53.34 0)
+			(effects
+				(font
+					(size 1.27 1.27)
+				)
+				(hide yes)
+			)
+		)
 		(pin "2"
 		)
@@
 		)
 		(property "Purchase-URL" ""
+			(at 110.49 78.74 0)
+			(effects
+				(font
+					(size 1.27 1.27)
+				)
+				(hide yes)
+			)
+		)
+		(property "Supplier" "Mouser"
 			(at 110.49 78.74 0)
 			(effects
@@
 			)
 		)
+		(property "Supplier" "Mouser"
+			(at 105.41 88.9 0)
+			(effects
+				(font
+					(size 1.27 1.27)
+				)
+				(hide yes)
+			)
+		)
 		(pin "26"
 		)
@@
 			)
 		)
+		(property "Supplier" "Mouser"
+			(at 92.71 36.83 0)
+			(effects
+				(font
+					(size 1.27 1.27)
+				)
+				(hide yes)
+			)
+		)
 		(pin "2"
 		)
@@
 			)
 		)
+		(property "Supplier" "Mouser"
+			(at 110.49 68.58 0)
+			(effects
+				(font
+					(size 1.27 1.27)
+				)
+				(hide yes)
+			)
+		)
 		(pin "2"
 		)
@@
 			(at 58.42 30.48 0)
 			(effects
+				(font
+					(size 1.27 1.27)
+				)
+				(hide yes)
+			)
+		)
+		(property "Supplier" "Mouser"
+			(at 58.42 30.48 0)
+			(effects
